Commit message: fix cloud creation and tf with normals

File: src/jaka_description/urdf/jaka_s12.urdf (robot description, URDF)
Before this commit: robot jaka_s12, 12 links, 11 joints
Links:
- added link camera_optical_frame
Joints:
- added joint camera_optical_joint: type fixed, parent camera_link, child camera_optical_frame, origin xyz=0 0 0 rpy=-1.5708 0 -1.5708

Commit message: real robot calibration jaka services bridge

File: src/jaka_description/urdf/jaka_s12.urdf (robot description, URDF)
Before this commit: robot jaka_s12, 13 links, 12 joints
Links:
- link camera_link: geometry collision box size=0.11 0.05 0.07; visual box size=0.11 0.05 0.07
Joints:
- joint camera_joint: origin xyz=0.0 0.1 0.07 rpy=-1.5708 -1.5708 0.0 -> xyz=0.00 0.115 0.07 rpy=-1.5708 -1.5708 0.0
- joint joint_1: limit lower=-1.58 upper=3.15 effort=2000 velocity=2.09 -> lower=-1.58 upper=4.7 effort=2000 velocity=2.09
- joint joint_6: limit lower=-6.28 upper=6.28 effort=1000 velocity=3.14 -> lower=-3.20 upper=3.20 effort=1000 velocity=3.14

Commit message: tray_pick_place OBB trays

File: src/jaka_description/urdf/jaka_s12.urdf (robot description, URDF)
Before this commit: robot jaka_s12, 13 links, 12 joints
Joints:
- joint camera_joint: origin xyz=0.00 0.115 0.07 rpy=-1.5708 -1.5708 0.0 -> xyz=0.00 0.115 0.08 rpy=-1.5708 -1.5708 0.0

Commit message: functioning pick from box movement opt

File: src/jaka_description/urdf/jaka_s12.urdf (robot description, URDF)
Before this commit: robot jaka_s12, 13 links, 12 joints
Joints:
- joint camera_joint: origin xyz=0.00 0.115 0.08 rpy=-1.5708 -1.5708 0.0 -> xyz=-0.02 0.115 0.08 rpy=-1.5708 -1.5708 0.0
